File: electronic_design/esp32_stepper_driver/esp32_stepper_driver.kicad_sch (KiCad schematic)
At the start: 15 parts

Commit message: finished design
Parts:
- removed C? (x2): C, symbol Device:C
- removed U?: AZ1117-3.3, symbol Regulator_Linear:AZ1117-3.3
- added J?: UART, symbol Connector:Screw_Terminal_01x04
- added J?: MOTOR, symbol Connector:Screw_Terminal_01x04
- added J?: INPUT, symbol Connector:Screw_Terminal_01x02
- added R? (x2): .5R, symbol Device:R
Connections:
- net VDD_5V is gone; now on net VDD5V: C?.1, C?.1, L?.2, R?.1
- net GND: now also U?.29 (GND), U?.8 (GND), J?.1 (Pin_1), J?.1 (Pin_1), R?.2, R?.2
- net VIN: now also U?.4 (Vs), J?.2 (Pin_2)
- net at U?.19 (D34): now also U?.1 (SENSE_A), R?.1
- net at U?.20 (D35): now also U?.15 (SENSE_B), R?.1
- net VDD5V: now reaches U?.30 (VIN)
- net VDD5V: now also U?.9 (Vss), J?.2 (Pin_2)
- net at U?.6 (RX2): now also J?.4 (Pin_4)
- net at U?.7 (TX2): now also J?.3 (Pin_3)
- net at U?.13 (OUT3): now also J?.3 (Pin_3)
- net at U?.14 (OUT4): now also J?.4 (Pin_4)
- net at U?.2 (OUT1): now also J?.1 (Pin_1)
- net at U?.3 (OUT2): now also J?.2 (Pin_2)
- net VDD_3V3: no longer names the net of U?.1 (3V3)
Other:
- note added: "MOTOR CONTROL"
- moved on the sheet: C?, D?, L?, R?, RV?, U?
